File: Hardware/Standard/ZigbeeLightController.sch (KiCad schematic (older format))
At the start: 97 parts, among them J1 M20-7870346, J2 1935268, J3 1935268, J4 1935161, Q1 2N7002, Q10 FDMS7682, Q11 FDMS7682, Q12 FDMS7682, Q13 FDMS7682, Q14 FDMS7682, Q2 2N7002, Q3 FDMS7682, Q4 FDMS7682, Q5 FDMS7682, Q6 FDMS7682, Q7 FDMS7682, Q8 FDMS7682, Q9 FDMS7682, SW1 SW_Push, U1 MCP16301, U10 ZXGD3009DY, U11 ZXGD3009DY, U12 ZXGD3009DY, U13 ZXGD3009DY, U14 ZXGD3009DY, U15 ZXGD3009DY, U16 ZXGD3009DY, U2 AP2120N-3.3, U3 JN5168-001-M00, U4 PCA9685, U5 ZXGD3009DY, U6 ZXGD3009DY, U7 ZXGD3009DY, U8 ZXGD3009DY, U9 ZXGD3009DY

Commit message: Standard hardware bugfixes: changed BOM to use correct 0603 part instead of 0402 part, widened pad for D3, changed R2 to 10k to reduce line item count, filling top layer
Parts:
- D3: footprint Diodes_SMD:D_0805 -> zll_lib:D_0805_LED
- R2: value 100k -> 10k
Changed lines of the file:
@@
 P 1200 7300
 F 0 "R2" V 1280 7300 50  0000 C CNN
-F 1 "100k" V 1100 7300 50  0000 C CNN
+F 1 "10k" V 1100 7300 50  0000 C CNN
 F 2 "Resistors_SMD:R_0603" V 1130 7300 50  0001 C CNN
 F 3 "" H 1200 7300 50  0001 C CNN
@@
 F 0 "D3" H 4250 8100 50  0000 C CNN
 F 1 "LED" H 4250 7900 50  0000 C CNN
-F 2 "Diodes_SMD:D_0805" H 4250 8000 50  0001 C CNN
+F 2 "zll_lib:D_0805_LED" H 4250 8000 50  0001 C CNN
 F 3 "" H 4250 8000 50  0001 C CNN
 	1    4250 8000
