File: Hardware/Mini/ZigbeeLightControllerMini.kicad_pcb (KiCad board)
At the start: 2 copper layers, 83 x 71 mm, 53 parts, among them J1 M20-7870346, J2 1935242, Q1 FDMS7682, Q2 FDMS7682, Q3 FDMS7682, Q4 FDMS7682, SW1 SW_Push, U1 MCP16301, U2 JN5168-001-M00, U3 AP2120N-3.3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

Commit message: Fixing PCB fill issue, using - and K for LED terminals
Other:
- board text added: "B -"
- board text added: "B K"
- board text added: "G -"
- board text added: "G K"
- board text added: "R -"
- board text added: "R K"
- board text added: "W -"
- board text added: "W K"
- board text removed: "BGND"
- board text removed: "BLED"
- board text removed: "GGND"
- board text removed: "GLED"
- board text removed: "RGND"
- board text removed: "RLED"
- board text removed: "WGND"
- board text removed: "WLED"
Changed lines of the file:
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@@
     (links 170)
     (no_connects 0)
-    (area 66.924999 26.424999 150.075001 97.575001)
+    (area 63.842857 26.424999 153.157143 97.879001)
     (thickness 1.6)
     (drawings 16)
@@
     (effects (font (size 1.5 1.5) (thickness 0.3)))
   )
-  (gr_text BLED (at 129 31 90) (layer F.SilkS)
+  (gr_text "B K" (at 129 31 90) (layer F.SilkS)
     (effects (font (size 1.5 1.5) (thickness 0.3)))
   )
-  (gr_text BGND (at 124 31 90) (layer F.SilkS)
+  (gr_text "B -" (at 124 31 90) (layer F.SilkS)
     (effects (font (size 1.5 1.5) (thickness 0.3)))
   )
-  (gr_text GLED (at 119 31 90) (layer F.SilkS)
+  (gr_text "G K" (at 119 31 90) (layer F.SilkS)
     (effects (font (size 1.5 1.5) (thickness 0.3)))
   )
-  (gr_text GGND (at 114 31 90) (layer F.SilkS)
+  (gr_text "G -" (at 114 31 90) (layer F.SilkS)
     (effects (font (size 1.5 1.5) (thickness 0.3)))
   )
-  (gr_text RLED (at 109 31 90) (layer F.SilkS)
+  (gr_text "R K" (at 109 31 90) (layer F.SilkS)
     (effects (font (size 1.5 1.5) (thickness 0.3)))
   )
-  (gr_text RGND (at 104 31 90) (layer F.SilkS)
+  (gr_text "R -" (at 104 31 90) (layer F.SilkS)
     (effects (font (size 1.5 1.5) (thickness 0.3)))
   )
-  (gr_text WLED (at 99 31 90) (layer F.SilkS)
+  (gr_text "W K" (at 99 31 90) (layer F.SilkS)
     (effects (font (size 1.5 1.5) (thickness 0.3)))
   )
-  (gr_text WGND (at 94 31 90) (layer F.SilkS)
+  (gr_text "W -" (at 94 31 90) (layer F.SilkS)
     (effects (font (size 1.5 1.5) (thickness 0.3)))
   )
